File: Hardware/schematic_tsc.sch (EAGLE design)
At the start: 105 parts, among them IC1 BQ25180YBGR, IC2 DRV2605YZFR, IC3 BMA423, IC9 RT6160AWSC, J1 503480-2400, J2 TC2030-IDC, J4 KH-TYPE-C-16P, Q1 20V/4.2A/52mΩ/1.4W, Q3 SI1308EDL-T1-GE3, U1 NRF52840_QF, U3 MAX17048G+T10, X1 32MHz, X2 32.768kHz

Commit message: Add files via upload
Parts:
- removed C32: 1uF, InkTime_v5:NORDIC_NRF_3_CAPACITOR_0402_L
- removed C34: 0.1uF, InkTime_v5:NORDIC_NRF_3_CAPACITOR_0402_L
- added C26, C28: 0.1uF, InkTime_v5:GRM011R60J152KE01L_2_GRM011R60J152KE01L
- C23, C24: device InkTime_v5:NORDIC_NRF_3_CAPACITOR_0402_L -> InkTime_v5:GRM011R60J152KE01L_2_GRM011R60J152KE01L
- renumbered U$32 to C33, U$33 to C25
Connections:
- net 3V3: now also C26.2; no longer C34.1
- net GND: now also C23.2, C26.1, C28.1; no longer C23.1, C32.2, C34.2
- net N$63: now also C28.2; no longer C32.1
- net VREG: now also C23.1; no longer C23.2
